File: WLEDController.kicad_sch (KiCad schematic)
At the start: 63 parts, among them J1 5V Power, J2 I2S EXTENSION, J3 LED Channel 1, J4 LED Channel 2, J5 LED Channel 3, J6 LED Channel 4, K1 SANYOU SRD, Q1 AOD403, Q2 IRLL2705, U1 AMS1117-3.3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

Commit message: Cleanup
Other:
- company: (none) -> Marc Schöndorf
- title: (none) -> WLED Controller
Changed lines of the file:
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@@
 	(generator_version "8.0")
 	(paper "A3")
+	(title_block
+		(title "WLED Controller")
+		(date "03.02.2025")
+		(rev "V1.0")
+		(company "Marc Schöndorf")
+	)
 	(junction
 		(at 223.52 90.17)

Commit message: Added Touch sensor
Parts:
- removed J2: I2S EXTENSION, Connector_IDC:IDC-Header_2x04_P2.54mm_Horizontal, symbol Connector_Generic:Conn_02x04_Odd_Even
- added J2: I2S Extension, Connector_IDC:IDC-Header_2x05_P2.54mm_Horizontal, symbol Connector_Generic:Conn_02x05_Odd_Even
- renumbered R4 to R3, R3 to R4
Connections:
- net +3.3V_D: now also J2.1 (Pin_1)
- net +5V_D: now also J2.2 (Pin_2)
- net BCK: now also J2.7 (Pin_7)
- net DOUT: now also J2.5 (Pin_5)
- net GND: now also J2.3 (Pin_3), J2.4 (Pin_4), J2.6 (Pin_6), J2.9 (Pin_9)
- net LRCK: now also J2.8 (Pin_8)
- net MCK: now also J2.10 (Pin_10)
- net at R3.1: now also U3.30 (IO_12/TDI); no longer U3.18 (IO_13/TCK)
- net at D1.2 (AK): now also U3.18 (IO_13/TCK); no longer U3.13 (IO_14/TMS)
- new net TOUCH: U3.13 (IO_14/TMS)
- no-connect marks 19 -> 18
Other:
- moved on the sheet: D1, R1, R2, R3, U2, U3
